File: hardware/hardware/logger.sch (EAGLE design)
At the start: 3 parts

Commit message: Basically finished schematic, should really include the eagle lbr in repo but that's effort...
Parts:
- added C1, C2, C3, C4, C5, C6, C7, C8: (no value), rcl:C-EU025_050-045X075
- added INPUTS: (no value), con-lstb:MA05-2
- added LED1, LED2: (no value), led:LED5MM
- added MCU: PIC18F4550_40, microchip:PIC18F4550_40
- added OPAMP1, OPAMP2: LM2902N, linear:LM2902N
- added R1, R10, R11, R12, R2, R5, R6, R7, R8, R9: 100R, rcl:R-EU_0207/10
- added R3, R4: 1KR, rcl:R-EU_0207/10
Connections:
- new net A0: MCU.RB0/AN12/INT0/LFT0/SDI/SDA, SRAM.A0
- new net A1: MCU.RB1/AN10/INT1/SCK/SCL, SRAM.A1
- new net A10: MCU.RD2/SPP2, SRAM.A10
- new net A11: MCU.RD3/SPP3, SRAM.A11
- new net A12: MCU.RD4/SPP4, SRAM.A12
- new net A13: MCU.RD5/SPP5/P1B, SRAM.A13
- new net A14: MCU.RD6/SPP6/P1C, SRAM.A14
- new net A15: MCU.RD7/SPP7/P1D, SRAM.A15
- new net A16: SRAM.A16
- new net A2: MCU.RB2/AN8/INT2/VMO, SRAM.A2
- new net A3: MCU.RB3/AN9/CCP2/VPO, SRAM.A3
- new net A4: MCU.RB4/AN11/KBI0/CSSPP, SRAM.A4
- new net A5: MCU.RB5/KBI1/PGM, SRAM.A5
- new net A6: MCU.RB6/KBI2/PGC, SRAM.A6
- new net A7: MCU.RB7/BKI3/PGD, SRAM.A7
- new net A8: MCU.RD0/SPP0, SRAM.A8
- new net A9: MCU.RD1/SPP1, SRAM.A9
- new net IP1: INPUTS.1, R8.2
- new net IP2: INPUTS.2, R7.2
- new net IP3: INPUTS.3, R6.2
- new net IP4: INPUTS.4, R5.2
- new net IP5: INPUTS.5, R12.2
- new net IP6: INPUTS.6, R11.2
- new net IP7: INPUTS.7, R10.2
- new net IP8: INPUTS.8, R9.2
- new net LEDA: MCU.RA0/AN0, R2.2
- new net LEDB: MCU.RA1/AN1, R1.2
- new net N$1: C1.1, OPAMP1D.-IN, R5.1
- new net N$10: C8.1, OPAMP2A.-IN, R12.1
- new net N$2: LED1.A, R1.1
- new net N$3: C4.1, OPAMP1C.-IN, R6.1
- new net N$4: LED2.A, R2.1
- new net N$5: C2.1, OPAMP1B.-IN, R7.1
- new net N$6: C3.1, OPAMP1A.-IN, R8.1
- new net N$7: C6.1, OPAMP2D.-IN, R9.1
- new net N$8: C5.1, OPAMP2C.-IN, R10.1
- new net N$9: C7.1, OPAMP2B.-IN, R11.1
- new net RAM_CE: MCU.RC1/T1OSI/ICCP2/!UOE, SRAM.CE
- new net RAM_CE2: MCU.RC6/TX/CK, SRAM.CE2
- new net RAM_OE: MCU.RC0/TIOSO/T13CKI, SRAM.OE
- new net RAM_WE: MCU.RC2/CCP1/P1A, SRAM.WE
- new net VREF: OPAMP1A.+IN, OPAMP1B.+IN, OPAMP1C.+IN, OPAMP1D.+IN, OPAMP2A.+IN, OPAMP2B.+IN, OPAMP2C.+IN, OPAMP2D.+IN, R3.1, R4.2
- net BUFFER_EN: now also MCU.RC7/RX/DT/SDO
- net CH1: now also OPAMP1A.OUT
- net CH2: now also OPAMP1B.OUT
- net CH3: now also OPAMP1C.OUT
- net CH4: now also OPAMP1D.OUT
- net CH5: now also OPAMP2A.OUT
- net CH6: now also OPAMP2B.OUT
- net CH7: now also OPAMP2C.OUT
- net CH8: now also OPAMP2D.OUT
- net GND: now also C1.2, C2.2, C3.2, C4.2, C5.2, C6.2, C7.2, C8.2, INPUTS.9, LED1.C, LED2.C, OPAMP1P.V-, OPAMP2P.V-, R4.1
- net SR_CLK: now also MCU.RE0/AN5/CK1SPP
- net SR_CLK_EN: now also MCU.RE1/AN6/CK2SPP
- net SR_PLOAD: now also MCU.RE2/AN7/OESPP
- net SR_SEROUT: now also MCU.RA2/AN2/VREF-/CVREF
- net VCC: now also OPAMP1P.V+, OPAMP2P.V+, R3.2
Other:
- note added: "1.0"
- note added: "CONNECTORS"
- note added: "Drawn by: Jon Sowman"
- note added: "NB: INVERTING"
- note added: "OPAMP PWR"
- note added: "SB3 - DATALOGGER"
- moved on the sheet: BUFFER, BUFFERP, SHIFTREG, SHIFTREGP, SRAM

Commit message: Nearly finished the schematic
Connections:
- net BUFO1 renamed D1
- net BUFO2 renamed D2
- net BUFO3 renamed D3
- net BUFO4 renamed D4
- net BUFO5 renamed D5
- net BUFO6 renamed D6
- net BUFO7 renamed D7
- net BUFO8 renamed D8
- net A0: now also MCU.RA3/AN3/VREF+; no longer MCU.RB0/AN12/INT0/LFT0/SDI/SDA
- net A1: now also MCU.RA4/T0CKI/CIOUT/RCV; no longer MCU.RB1/AN10/INT1/SCK/SCL
- net A2: now also MCU.RA5/AN4/!SS!/HLVDIN/C2OUT; no longer MCU.RB2/AN8/INT2/VMO
- net CH1: now also MCU.RB0/AN12/INT0/LFT0/SDI/SDA
